File: Breakout_board/FDC1004_V1/FDC1004_v1.kicad_pcb (KiCad board)
At the start: 2 copper layers, 30 x 27.5 mm, 10 parts, among them J1 CONUFL001-SMD-T, J2 CONUFL001-SMD-T, J3 CONUFL001-SMD-T, J4 CONUFL001-SMD-T, J5 Conn_01x02, U1 FDC1004QDGSRQ1, U2 Adafruit QT Py ESP32-S3, U3 MCP9701T-E/TT

Commit message: update board files
Parts:
- added J6: Conn_01x04, Connector_PinHeader_2.54mm:PinHeader_1x04_P2.54mm_Vertical, F.Cu at (108.4, 67.0)
- added R3: RMCF1206JT1K80, FDC1004_Footprints:STA_RMCF1206_STC, F.Cu at (99.0, 88.5)
- added R4: RMCF1206JT1K80, FDC1004_Footprints:STA_RMCF1206_STC, F.Cu at (98.5, 72.0)
Connections:
- J1 pad 3: GND -> /drive
- J2 pad 3: GND -> /drive
- J3 pad 2: GND -> /drive
- J4 pad 2: GND -> /drive
- U1 pad 1: unconnected-(U1-SHLD1-Pad1) -> /shield
Routing:
- net GND: track 270.6 -> 179.2 mm, vias 2 -> 1
- net /drive: track 0.00 -> 88.6 mm
- net /shield: track 0.00 -> 8.65 mm
Other:
- board text added: "Act shield"
- board text added: "FDC1004 Cap Breakout Board V1"
- board text added: "GND shield"
- board text added: "PARSES Lab K.Dorsey@ Northeastern"
- board text removed: "FDC1004 Cap Meas Board V1 K.Dorsey@Northeastern.edu"
