File: Breakout_board/FDC1004_V1/FDC1004_v1.kicad_sch (KiCad schematic)
At the start: 10 parts, among them J1 CONUFL001-SMD-T, J2 CONUFL001-SMD-T, J3 CONUFL001-SMD-T, J4 CONUFL001-SMD-T, J5 Conn_01x02, U1 FDC1004QDGSRQ1, U2 Adafruit QT Py ESP32-S3, U3 MCP9701T-E/TT

Commit message: update board files
Parts:
- added J6: Conn_01x04, Connector_PinHeader_2.54mm:PinHeader_1x04_P2.54mm_Vertical, symbol Connector_Generic:Conn_01x04
- added R3, R4: RMCF1206JT1K80, FDC1004_Footprints:STA_RMCF1206_STC, symbol FDC1004Lib:RMCF1206JT1K80
Connections:
- net GND: now also J6.1 (Pin_1), J6.2 (Pin_2), J6.3 (Pin_3), J6.4 (Pin_4), R3.2; no longer J1.3, J2.3, J3.2, J4.2
- net shield: now reaches U1.1 (SHLD1)
- net shield: now also R4.2
- new net drive: J1.3, J2.3, J3.2, J4.2, R3.1, R4.1
- no-connect marks 15 -> 14
